Commit message: updates

File: my-robot/robot.urdf (robot description, URDF)
Before this commit: robot onshape, 11 links, 10 joints
Links:
- removed link base_link
- removed link left_foot
- removed link right_foot
- added link foot, mass 0.06548220204090636487; collision mesh filename=package:///foot.stl; visual mesh filename=package:///foot.stl
- added link foot_2, mass 0.06548220204090636487; collision mesh filename=package:///foot.stl; visual mesh filename=package:///foot.stl
- added link main_body, mass 0.54025647521951047914; collision mesh filename=package:///base_link.stl; collision mesh filename=package:///st3125.stl
- link left_lower_hip: mass 0.073736344590716929037 -> 0.079411681455473101532
- link left_lower_leg: mass 0.08014448865577621095 -> 0.089161262608861993617; geometry collision mesh filename=package:///hip_servo_knee_link.stl; collision mesh filename=package:///st3125.stl
- link left_upper_hip: mass 0.074496678806569724407 -> 0.080172015671325883024
- link left_upper_leg: mass 0.08014448865577621095 -> 0.089161262608861993617; geometry collision mesh filename=package:///hip_servo_knee_link.stl; collision mesh filename=package:///st3125.stl
- link right_lower_hip: mass 0.073736344590716929037 -> 0.079411681455473101532
- link right_lower_leg: mass 0.08014448865577621095 -> 0.089161262608861993617; geometry collision mesh filename=package:///hip_servo_knee_link.stl; collision mesh filename=package:///st3125.stl
- link right_upper_hip: mass 0.074496678806569724407 -> 0.080172015671325883024
- link right_upper_leg: mass 0.08014448865577621095 -> 0.089161262608861993617; geometry collision mesh filename=package:///hip_servo_knee_link.stl; collision mesh filename=package:///st3125.stl
Joints:
- removed joint Left_Foot
- removed joint Left_Hip
- removed joint Left_Hip_Around_Z
- removed joint Left_Hip_In_Out
- removed joint Left_Knee
- removed joint Right_Foot
- removed joint Right_Hip
- removed joint Right_Hip_Around_Z
- removed joint Right_Hip_In_Out
- removed joint Right_Knee
- added joint left_foot: type revolute, parent left_lower_leg, child foot, origin xyz=-0.099999999999999908407 1.3877787807814456755e-17 -3.9999999999991431299e-05 rpy=-1.5777218104420257128e-30 -1.0924123923090688949e-46 0, axis 0 0 1, limit lower=-1.2217304763960306069 upper=1.2217304763960306069 effort=1 velocity=20
- added joint left_hip: type revolute, parent left_lower_hip, child left_upper_leg, origin xyz=0.018683161360494256187 0.049999999999999940326 0.017650000000000005962 rpy=1.5707963267948958919 -2.7755575615629071283e-16 -1.570796326794896558, axis 0 0 1, limit lower=-1.2217304763960306069 upper=1.2217304763960306069 effort=1 velocity=20
- added joint left_hip_around_torso: type revolute, parent main_body, child left_upper_hip, origin xyz=-0.02159616091652009906 0.069551495045236888526 0.099239393956395111074 rpy=-3.141592653589793116 -2.775557561562669977e-16 -5.7211887260545391184e-18, axis 0 0 1, limit lower=-0.34906585039886589561 upper=0.34906585039886589561 effort=1 velocity=20
- added joint left_in_out: type revolute, parent left_upper_hip, child left_lower_hip, origin xyz=0.029362999556025719261 0.017926838639505858486 0.039425000000000022526 rpy=1.570796326794891673 -2.77555756156270942e-16 -8.3838845719492212933e-16, axis 0 0 1, limit lower=-0.1745329251994329478 upper=0.1745329251994329478 effort=1 velocity=20
- added joint left_knee: type revolute, parent left_upper_leg, child left_lower_leg, origin xyz=-0.10000000000000008882 2.7755575615628913511e-17 -3.9999999999998370193e-05 rpy=-4.203895392974408274e-45 1.092412392309106233e-46 0, axis 0 0 1, limit lower=-2.4434609527920612138 upper=2.4434609527920612138 effort=1 velocity=20
- added joint right_foot: type revolute, parent right_lower_leg, child foot_2, origin xyz=-0.099999999999999408806 1.249000902703301108e-16 -4.000000000001224798e-05 rpy=-6.2975486165559455013e-17 -6.2785316187098858277e-32 -7.0997481469891062487e-30, axis 0 0 1, limit lower=-1.2217304763960306069 upper=1.2217304763960306069 effort=1 velocity=20
- added joint right_hip: type revolute, parent right_lower_hip, child right_upper_leg, origin xyz=0.018683161360494193737 -0.050000000000000002776 0.018450000000000021938 rpy=-1.57079632679489678 7.8886090522101180541e-30 1.570796326794896558, axis 0 0 1, limit lower=-1.2217304763960306069 upper=1.2217304763960306069 effort=1 velocity=20
- added joint right_hip_around_torso: type revolute, parent main_body, child right_upper_hip, origin xyz=-0.12640383908348010178 0.069551495045236791381 0.099239393956395305363 rpy=3.141592653589793116 7.703719777548948886e-33 -3.141592653589793116, axis 0 0 1, limit lower=-0.34906585039886589561 upper=0.34906585039886589561 effort=1 velocity=20
- added joint right_in_out: type revolute, parent right_upper_hip, child right_lower_hip, origin xyz=0.029362999556025615178 -0.018283161360493918601 0.039425000000000237632 rpy=-1.5707963267949018871 -6.7649150867249521185e-29 -1.3921856581593558197e-14, axis 0 0 1, limit lower=-0.1745329251994329478 upper=0.1745329251994329478 effort=1 velocity=20
- added joint right_knee: type revolute, parent right_upper_leg, child right_lower_leg, origin xyz=-0.099999999999999686362 4.1633363423443370266e-17 -3.9999999999984492405e-05 rpy=3.5219910549969984548e-17 -8.4077907859489024255e-45 -7.8886090522101180541e-31, axis 0 0 1, limit lower=-2.4434609527920612138 upper=2.4434609527920612138 effort=1 velocity=20
